File: pcb/emmon.sch (KiCad schematic (older format))
At the start: 48 parts, among them J1 PROG_CONN, J2 ANT_CONN, J3 AC_CONN, Q1 PT11-21C/L41/TR8, U1 DS3231SN, U2 CAT24C32WI-GT3, U3 LM393DR2G, U4 ESP-12E, U5 Ai-Thinker-Ra-01

Commit message: se aplican las correciones de la revisión del profesor
Parts:
- U3: Description (none) -> Analog Comparators 2V - 36V, ±1V ~ 18V SOIC-8_150mil RoHS; LCSC (none) -> C7955
Changed lines of the file:
@@
 F 2 "Package_SO:SOIC-8_3.9x4.9mm_P1.27mm" H 8850 3100 50  0001 C CNN
 F 3 "https://datasheet.lcsc.com/szlcsc/ON-Semicon-ON-LM393DR2G_C7955.pdf" H 8850 3100 50  0001 C CNN
+F 4 "C7955" H 8850 3100 50  0001 C CNN "LCSC"
+F 5 "Analog Comparators 2V - 36V, ±1V ~ 18V SOIC-8_150mil RoHS" H 8850 3100 50  0001 C CNN "Description"
 	3    8850 3100
 	1    0    0    -1
